File: 4040.kicad_pcb (KiCad board)
At the start: 2 copper layers, 281.3 x 76.5 mm, 127 parts, among them J1 USB_C_Receptacle_USB2.0_16P, SW1 SW_Push, U2 ATmega32U4-A, Y1 16MHz

Commit message: main
Parts:
- added U1: USBLC6-2SC6, Package_TO_SOT_SMD:SOT-23-6, B.Cu at (67.9, 89.2)
- moved F2 1.20 mm to (68.2, 85.6)
Connections:
- J1 pad A6: D+ -> A+
- J1 pad A7: D- -> A-
- J1 pad B6: D+ -> A+
- J1 pad B7: D- -> A-
Routing:
- net GND: track 654.4 -> 672.5 mm
- net D+: track 24.5 -> 16.4 mm
- net D-: track 22.9 -> 16.0 mm
- net A+: track 0.00 -> 5.79 mm
- net A-: track 0.00 -> 5.75 mm
- net VCC: track 12.6 -> 16.6 mm
- net +5V: track 672.9 -> 674.2 mm, vias 2 -> 4
Other:
- board size 281.3 x 76.5 mm -> 281.7 x 77 mm

Commit message: update
Parts:
- moved SW1 0.16 mm to (183.9, 140.5)
Routing:
- net Net-(HL5-DOUT): track 123.2 -> 120.2 mm
- net COL9: track 118.1 -> 119.1 mm
- net COL10: track 143.5 -> 144.5 mm
- net +5V: track 674.2 -> 673.4 mm
- net COL11: track 169.0 -> 169.7 mm
- net Net-(HL3-DOUT): track 63.1 -> 62.5 mm
Other:
- outline, holes or cut-outs redrawn
- board text added: "Designed by LexR V1.1"
